File: fs-a1gt/turbo-r-1mb/turbo-r-1mb.kicad_sch (KiCad schematic)
At the start: 18 parts, among them U1 220-1-20-003, U2 220-1-20-003, U3 KM44C1000, U4 SN74LS670D, U5 CD74HCT367M96, U6 CD74HCT30M96, U7 SN74HCT32DR, U8 KM44C1000

Commit message: PCB ready for ordering
Parts:
- added C1, C2, C3, C4: 100nF, Capacitor_SMD:C_0603_1608Metric, symbol Device:C_Small
- TP1: value D6 -> D5
- TP10: value nIORD -> ~{IORD}
- TP7: value nA[3/5/6/7] -> A3,5,6,7
- TP8: value nIOWR -> ~{IOWR}
- U1: renamed from U6; value CD74HCT30M96 -> CD74HCT30
- U3: renamed from U4; footprint Package_SO:SOIC-16W_5.3x10.2mm_P1.27mm -> Package_SO:SOIC-16_3.9x9.9mm_P1.27mm
- U4: renamed from U5; value CD74HCT367M96 -> CD74HCT367
- renumbered U3 to IC1, U8 to IC2, U1 to IC38, U2 to IC40, U7 to U2
Connections:
- net GND: now also C1.2, C2.2, C3.2, C4.2
- net VCC: now also C1.1, C2.1, C3.1, C4.1
